File: stm32 PCB design.kicad_pcb (KiCad board)
At the start: 2 copper layers, 44.2 x 31.3 mm, 32 parts, among them J1 USB_B_Micro, J2 Conn_01x04_Pin, J3 Conn_01x04_Pin, J4 Conn_01x04_Pin, SW2 SW_SPDT, U1 STM32F103C8T6, U2 AMS1117, Y1 16MHz

Commit message: Documentation updated and design rule checks validated
Parts:
- moved J3 19.1 mm to (112.0, 35.0)
- moved J2 14.1 mm to (129.4, 34.8)
- moved R2 4.93 mm to (104.2, 42.2), turned to -90 degrees
- moved R3 3.20 mm to (123.0, 47.0), turned to -90 degrees
- moved J1 1.88 mm to (136.6, 48.0)
- moved C5 1.21 mm to (115.0, 54.8), turned to 180 degrees
- moved R4 1.02 mm to (111.3, 58.0), turned to 180 degrees
- moved C4 0.98 mm to (106.5, 45.8)
- moved C7 0.22 mm to (109.8, 43.0)
- moved C12 0.18 mm to (105.2, 48.3)
- turned C10 to 180 degrees
- turned C9 to 180 degrees
- turned C6 to -90 degrees
Connections:
- C1 pad 2: <NO NET> -> GND
- C10 pad 2: <NO NET> -> GND
- C11 pad 2: <NO NET> -> GND
- C12 pad 2: <NO NET> -> GND
- C13 pad 1: /HSE_IN -> /HSE_OUT
- C13 pad 2: <NO NET> -> GND
- C2 pad 2: <NO NET> -> GND
- C3 pad 2: <NO NET> -> GND
- C4 pad 2: <NO NET> -> GND
- C5 pad 2: <NO NET> -> GND
- C6 pad 2: <NO NET> -> GND
- C7 pad 2: <NO NET> -> GND
- C8 pad 2: <NO NET> -> GND
- C9 pad 2: <NO NET> -> GND
- J1 pad 5: <NO NET> -> GND
- J2 pad 4: <NO NET> -> GND
- J3 pad 4: <NO NET> -> GND
- J4 pad 4: <NO NET> -> GND
- R1 pad 2: <NO NET> -> GND
- SW2 pad 3: <NO NET> -> GND
- U1 pad 23: <NO NET> -> GND
- U1 pad 35: <NO NET> -> GND
- U1 pad 47: <NO NET> -> GND
- U1 pad 6: /HSE_IN -> /HSE_OUT
- U1 pad 8: <NO NET> -> GND
- U2 pad 1: <NO NET> -> GND
- Y1 pad 2: /HSE_IN -> GND
- Y1 pad 3: /HSE_IN -> /HSE_OUT
- Y1 pad 4: /HSE_IN -> GND
Routing:
- net +3.3V: track 0.00 -> 149.3 mm, vias 0 -> 6
- net GND: track 0.00 -> 36.4 mm, vias 0 -> 22
- net /SW_DIO: track 0.00 -> 19.1 mm
- net /USB_D-: track 0.00 -> 18.0 mm
- net /USB_D+: track 0.00 -> 17.9 mm
- net /BOOT0: track 0.00 -> 14.6 mm
- net /SWCLK: track 0.00 -> 14.5 mm
- net /USART1_RX: track 0.00 -> 12.7 mm
- net /USART1_TX: track 0.00 -> 11.2 mm
- net /I2C2_SCL: track 0.00 -> 10.8 mm
- net /I2C2_SDA: track 0.00 -> 10.2 mm
- net /NRST: track 0.00 -> 10.1 mm
- net /HSE_IN: track 0.00 -> 8.12 mm
- net +3.3VA: track 0.00 -> 5.84 mm
- net /HSE_OUT: track 0.00 -> 5.46 mm
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- added copper zone on F.Cu, net +3.3V
- added copper zone on B.Cu, net GND
- added copper zone on F.Cu, net GND
- added copper zone on F.Cu, net VBUS
Other:
- board text added: "BOOT"
- board text added: "I2C"
- board text added: "SWD"
- board text added: "UART"
- board text added: "USB"
